File: Hardware/Qwiic_AS3935_Lightning_Detector.brd (EAGLE design)
At the start: 25.4 x 25.4 mm, 67 parts, among them U1 AS3935

Commit message: Library update, small changeds to PCB
Parts:
- removed U$42: (no value), Labels:MISO-[)-03
- added U$11: (no value), Labels:CS#-<]-04
- U$13: device Labels:MOSI-[)-03 -> Labels:MISO-(]-03
- U$14: device Labels:MOSI-[)-03 -> INT:INT0
- U$15: device Labels:SCK-[)-03 -> INT_2:INT0
- U$16: device Labels:SCK-[)-03 -> Labels:MOSI-(]-03
- U$19, U$23: device INT:INT0 -> Labels:SCK-(]-03
- U$22: device INT:INT0 -> Labels:MOSI-(]-03
- U$24: device INT:INT0 -> INT_2:INT0
- U$29: device CS:#CS0 -> INT:INT0
- U$30: device CS:#CS0 -> CS_2:#CS0
- moved U$15 22.2 mm to (17.8, 23.7), turned to 270 degrees
- moved U$23 18.8 mm to (17.8, 4.95)
- moved U$29 10.7 mm to (20.3, 4.83), turned to 270 degrees
- moved U$22 6.51 mm to (15.2, 5.59), turned to 270 degrees
- moved U$14 6.06 mm to (20.3, 4.83), turned to 270 degrees
- moved U$13 4.79 mm to (12.7, 5.59), turned to 270 degrees
- moved U$16 4.79 mm to (15.2, 5.59), turned to 270 degrees
- moved U$19 4.27 mm to (17.8, 4.95), turned to 270 degrees
- moved U$10 4.19 mm to (5.08, 5.71), turned to 270 degrees
- moved U$9 4.19 mm to (5.08, 5.71), turned to 270 degrees
- moved U$17 4.06 mm to (7.62, 5.46), turned to 270 degrees
- moved U$18 4.06 mm to (7.62, 5.46), turned to 270 degrees
- moved U$30 3.43 mm to (10.2, 4.83), turned to 270 degrees
Routing:
- net GND: track 14.6 -> 18.7 mm, vias 12 -> 10
- net N$4: track 8.13 -> 7.04 mm
