File: Hardware/Qwiic_AS3935_Lightning_Detector.brd (EAGLE design)
At the start: 25.4 x 25.4 mm, 67 parts, among them U1 AS3935

Commit message: Fixed AS3935 SKU in library
Parts:
- R7: value 10 -> 10k
Changed lines of the file:
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@@
 <layer number="115" name="ReferenceISLANDS" color="7" fill="1" visible="no" active="no"/>
 <layer number="116" name="Patch_BOT" color="9" fill="4" visible="no" active="no"/>
-<layer number="117" name="PM_Ref" color="26" fill="1" visible="no" active="yes"/>
+<layer number="117" name="PM_Ref" color="26" fill="1" visible="yes" active="yes"/>
 <layer number="118" name="Rect_Pads" color="7" fill="1" visible="no" active="no"/>
-<layer number="119" name="PF_Ref" color="31" fill="1" visible="no" active="yes"/>
-<layer number="120" name="WFL_Ref" color="25" fill="1" visible="no" active="yes"/>
+<layer number="119" name="PF_Ref" color="31" fill="1" visible="yes" active="yes"/>
+<layer number="120" name="WFL_Ref" color="25" fill="1" visible="yes" active="yes"/>
 <layer number="121" name="_tsilk" color="7" fill="1" visible="no" active="no"/>
 <layer number="122" name="_bsilk" color="7" fill="1" visible="no" active="no"/>
@@
 <attribute name="VALUE" x="14.859" y="7.366" size="0.6096" layer="27" font="vector" ratio="20" rot="R270" align="top-center"/>
 </element>
-<element name="R7" library="SparkFun-Resistors" package="0603" value="10" x="18.542" y="12.7" smashed="yes" rot="R270">
+<element name="R7" library="SparkFun-Resistors" package="0603" value="10k" x="18.542" y="12.7" smashed="yes" rot="R270">
 <attribute name="NAME" x="19.304" y="12.7" size="0.6096" layer="25" font="vector" ratio="20" rot="R270" align="bottom-center"/>
-<attribute name="PROD_ID" value="RES-12581" x="18.542" y="12.7" size="1.778" layer="27" font="vector" ratio="15" rot="R270" display="off"/>
-<attribute name="VALUE" value="10" x="17.78" y="12.7" size="0.6096" layer="27" font="vector" ratio="20" rot="R270" align="top-center"/>
+<attribute name="PROD_ID" value="RES-00824" x="18.542" y="12.7" size="1.778" layer="27" font="vector" ratio="15" rot="R270" display="off"/>
+<attribute name="VALUE" value="10k" x="17.78" y="12.7" size="0.6096" layer="27" font="vector" ratio="20" rot="R270" align="top-center"/>
 </element>
 <element name="JP4" library="SparkFun-Jumpers" package="SMT-JUMPER_3_2-NC_TRACE_SILK" value="JUMPER-SMT_3_2-NC_TRACE_SILK" x="12.7" y="6.731" smashed="yes" rot="MR180">
@@
 <element name="U1" library="temp_parts" package="16LD_MLPQ" value="AS3935" x="12.7" y="12.7" smashed="yes" rot="R180">
 <attribute name="NAME" x="15.24" y="16.002" size="0.6096" layer="25" font="vector" ratio="15" rot="R180"/>
-<attribute name="PROD_ID" value="IC-11133" x="12.7" y="12.7" size="1.778" layer="27" font="vector" ratio="15" rot="R180" display="off"/>
+<attribute name="PROD_ID" value="IC-11333" x="12.7" y="12.7" size="1.778" layer="27" font="vector" ratio="15" rot="R180" display="off"/>
 <attribute name="VALUE" x="15.24" y="9.525" size="0.6096" layer="27" font="vector" ratio="15" rot="R180"/>
 </element>

Commit message: Version x02 Exposed pad underneath was not connected to ground, coil package was incorrect.
Routing:
- net GND: track 18.7 -> 25.6 mm, vias 10 -> 11
- net INP: track 11.7 -> 12.5 mm
Other:
- board text added: "x02"
- board text removed: "x01"
Changed lines of the file:
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@@
 <wire x1="0" y1="25.4" x2="0" y2="0" width="0.2032" layer="20"/>
 <text x="20.447" y="-10.287" size="1.778" layer="51" font="vector">Elias Santistevan</text>
-<text x="23.368" y="1.143" size="1.27" layer="16" font="vector" rot="MR0" align="center">x01</text>
+<text x="23.368" y="1.143" size="1.27" layer="16" font="vector" rot="MR0" align="center">x02</text>
 </plain>
 <attributes>
@@
 <via x="1.651" y="12.954" extent="1-16" drill="0.3048"/>
 <contactref element="L1" pad="2"/>
-<wire x1="23.114" y1="14.224" x2="23.114" y2="17.018" width="0.508" layer="1"/>
+<wire x1="23.114" y1="14.224" x2="23.114" y2="17.477" width="0.508" layer="1"/>
 <via x="11.176" y="19.685" extent="1-16" drill="0.3048"/>
 <contactref element="U1" pad="4"/>
@@
 <wire x1="17.653" y1="6.731" x2="17.78" y2="6.604" width="0.2032" layer="16"/>
 <wire x1="17.78" y1="6.604" x2="17.78" y2="5.461" width="0.2032" layer="16"/>
+<wire x1="12.7066" y1="12.7066" x2="12.3816" y2="13.0316" width="0.254" layer="1"/>
+<wire x1="12.3816" y1="13.0316" x2="12.3816" y2="13.208" width="0.254" layer="1"/>
+<wire x1="12.3816" y1="13.208" x2="12.3816" y2="14.6166" width="0.254" layer="1"/>
+<wire x1="12.7066" y1="12.7066" x2="13.0316" y2="12.3816" width="0.254" layer="1"/>
+<wire x1="13.0316" y1="12.3816" x2="14.6186" y2="12.3816" width="0.254" layer="1"/>
+<wire x1="14.6186" y1="13.6816" x2="12.8552" y2="13.6816" width="0.254" layer="1"/>
+<wire x1="12.8552" y1="13.6816" x2="12.3816" y2="13.208" width="0.254" layer="1"/>
+<via x="15.494" y="14.351" extent="1-16" drill="0.3048"/>
 </signal>
 <signal name="3.3V">
@@
 <wire x1="9.779" y1="14.859" x2="8.763" y2="13.843" width="0.2032" layer="16"/>
 <wire x1="8.763" y1="13.843" x2="8.763" y2="12.192" width="0.2032" layer="16"/>
-<wire x1="13.6525" y1="2.9845" x2="12.0015" y2="2.9845" width="0.2032" layer="16"/>
+<wire x1="13.6525" y1="2.9845" x2="11.2395" y2="2.9845" width="0.2032" layer="16"/>
 <contactref element="U1" pad="13"/>
 <wire x1="11.7316" y1="10.7926" x2="11.7316" y2="9.9536" width="0.2032" layer="1"/>
 <wire x1="11.7316" y1="9.9536" x2="11.303" y2="9.525" width="0.2032" layer="1"/>
-<wire x1="12.0015" y1="2.9845" x2="9.271" y2="5.715" width="0.2032" layer="16"/>
+<wire x1="11.2395" y1="2.9845" x2="9.271" y2="4.953" width="0.2032" layer="16"/>
 <wire x1="9.271" y1="7.747" x2="9.398" y2="7.874" width="0.2032" layer="16"/>
-<wire x1="9.271" y1="7.747" x2="9.271" y2="5.715" width="0.2032" layer="16"/>
+<wire x1="9.271" y1="7.747" x2="9.271" y2="4.953" width="0.2032" layer="16"/>
 <via x="9.398" y="7.874" extent="1-16" drill="0.3048"/>
 <wire x1="8.763" y1="12.192" x2="10.795" y2="12.192" width="0.2032" layer="16"/>
@@
 <signal name="MISO">
 <contactref element="J4" pad="4"/>
-<wire x1="12.7" y1="1.143" x2="12.7" y2="1.397" width="0.2032" layer="16"/>
 <contactref element="U1" pad="12"/>
 <wire x1="10.7916" y1="11.7316" x2="9.9536" y2="11.7316" width="0.2032" layer="1"/>
@@
 <wire x1="8.763" y1="10.541" x2="8.89" y2="10.668" width="0.2032" layer="16"/>
 <via x="8.89" y="10.668" extent="1-16" drill="0.3048"/>
-<wire x1="12.7" y1="1.397" x2="8.763" y2="5.334" width="0.2032" layer="16"/>
-<wire x1="8.763" y1="5.334" x2="8.763" y2="10.541" width="0.2032" layer="16"/>
+<wire x1="12.7" y1="1.143" x2="12.319" y2="1.143" width="0.2032" layer="16"/>
+<wire x1="12.319" y1="1.143" x2="8.763" y2="4.699" width="0.2032" layer="16"/>
+<wire x1="8.763" y1="4.699" x2="8.763" y2="10.541" width="0.2032" layer="16"/>
 </signal>
 <signal name="SCLK/SCL">
@@
 <wire x1="17.614" y1="11.85" x2="16.4324" y2="13.0316" width="0.254" layer="1"/>
 <contactref element="L1" pad="1"/>
-<wire x1="23.114" y1="11.176" x2="23.114" y2="9.017" width="0.508" layer="1"/>
+<wire x1="23.114" y1="11.176" x2="23.114" y2="8.177" width="0.508" layer="1"/>
 <contactref element="U1" pad="3"/>
 <wire x1="16.4324" y1="13.0316" x2="14.6186" y2="13.0316" width="0.254" layer="1"/>

Commit message: One more time
Parts:
- moved FRAME1 8.98 mm to (-7.62, -19.1)
Routing:
- net GND: track 25.6 -> 22.7 mm
Changed lines of the file:
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@@
 <wire x1="25.4" y1="25.4" x2="0" y2="25.4" width="0.2032" layer="20"/>
 <wire x1="0" y1="25.4" x2="0" y2="0" width="0.2032" layer="20"/>
-<text x="20.447" y="-10.287" size="1.778" layer="51" font="vector">Elias Santistevan</text>
+<text x="19.177" y="-19.177" size="1.778" layer="51" font="vector">Elias Santistevan</text>
 <text x="23.368" y="1.143" size="1.27" layer="16" font="vector" rot="MR0" align="center">x02</text>
 </plain>
@@
 </autorouter>
 <elements>
-<element name="FRAME1" library="SparkFun-Aesthetics" package="CREATIVE_COMMONS" value="FRAME-LETTER" x="-6.35" y="-10.16" smashed="yes">
-<attribute name="DESIGNER" value="" x="-6.35" y="-10.16" size="1.778" layer="27" display="off"/>
-<attribute name="REV" value="" x="-6.35" y="-10.16" size="1.778" layer="27" display="off"/>
+<element name="FRAME1" library="SparkFun-Aesthetics" package="CREATIVE_COMMONS" value="FRAME-LETTER" x="-7.62" y="-19.05" smashed="yes">
+<attribute name="DESIGNER" value="" x="-7.62" y="-19.05" size="1.778" layer="27" display="off"/>
+<attribute name="REV" value="" x="-7.62" y="-19.05" size="1.778" layer="27" display="off"/>
 </element>
 <element name="J1" library="SparkFun-Connectors" package="1X04_1MM_RA" value="" x="5.08" y="12.7" smashed="yes" rot="R270">
@@
 <wire x1="12.7066" y1="12.7066" x2="12.3816" y2="13.0316" width="0.254" layer="1"/>
 <wire x1="12.3816" y1="13.0316" x2="12.3816" y2="13.208" width="0.254" layer="1"/>
-<wire x1="12.3816" y1="13.208" x2="12.3816" y2="14.6166" width="0.254" layer="1"/>
 <wire x1="12.7066" y1="12.7066" x2="13.0316" y2="12.3816" width="0.254" layer="1"/>
-<wire x1="13.0316" y1="12.3816" x2="14.6186" y2="12.3816" width="0.254" layer="1"/>
 <wire x1="14.6186" y1="13.6816" x2="12.8552" y2="13.6816" width="0.254" layer="1"/>
 <wire x1="12.8552" y1="13.6816" x2="12.3816" y2="13.208" width="0.254" layer="1"/>
